File: 4-bit-pincode.kicad_sch (KiCad schematic)
At the start: 0 parts

Commit message: Complete schematic
Parts:
- added C1: 104, Capacitor_THT:C_Disc_D5.0mm_W2.5mm_P2.50mm, symbol Device:C
- added D1, D2: 1N4007, Diode_THT:D_DO-41_SOD81_P7.62mm_Horizontal, symbol Device:D
- added D3: LED_GREEN, LED_THT:LED_D5.0mm, symbol Device:LED
- added D4: LED_RED, LED_THT:LED_D5.0mm, symbol Device:LED
- added Q1, Q2, Q3, Q4: PN2222A, Package_TO_SOT_THT:TO-92_Inline, symbol Transistor_BJT:PN2222A
- added R1, R2, R3: 10k, Resistor_THT:R_Axial_DIN0207_L6.3mm_D2.5mm_P7.62mm_Horizontal, symbol Device:R
- added R10: 1k, Resistor_THT:R_Axial_DIN0207_L6.3mm_D2.5mm_P7.62mm_Horizontal, symbol Device:R
- added R4, R5, R6, R7: 5.1k, Resistor_THT:R_Axial_DIN0207_L6.3mm_D2.5mm_P7.62mm_Horizontal, symbol Device:R
- added R8, R9: 220, Resistor_THT:R_Axial_DIN0207_L6.3mm_D2.5mm_P7.62mm_Horizontal, symbol Device:R
- added SW1, SW2, SW3, SW4, SW5: SW_Push, Button_Switch_THT:SW_PUSH_6mm, symbol Switch:SW_Push
- added U1: 74HC595, Package_DIP:DIP-16_W7.62mm, symbol 74xx:74HC595
Connections:
- new net: Q3.2 (B), R6.1
- new net: R6.2, U1.2 (QC)
- new net: R1.2, SW5.2, U1.10 (~{SRCLR})
- new net: Q2.1 (E), SW3.1
- new net: Q2.2 (B), R5.1
- new net: C1.1, D2.1 (K), R2.1, SW2.2, SW3.2, SW4.2, U1.11 (SRCLK), U1.12 (RCLK)
- new net: D4.1 (K), R9.1
- new net: Q1.2 (B), R4.1
- new net: R4.2, U1.15 (QA)
- new net: D1.1 (K), R3.1, U1.14 (SER)
- new net: D1.2 (A), D2.2 (A), SW1.1
- new net: D3.1 (K), R8.1
- new net: D3.2 (A), R7.1, U1.3 (QD)
- new net: R5.2, U1.1 (QB)
- new net: Q1.1 (E), SW2.1
- new net: D4.2 (A), Q4.3 (C), R10.1
- new net: Q3.1 (E), SW4.1
- new net: Q4.2 (B), R7.2
- new net +5V: Q1.3 (C), Q2.3 (C), Q3.3 (C), R1.1, R10.2, SW1.2, U1.16 (VCC)
- new net GND: C1.2, Q4.1 (E), R2.2, R3.2, R8.2, R9.2, SW5.1, U1.13 (~{OE}), U1.8 (GND)
- no-connect marks 0 -> 5
